File: Hardware/pRadio_HW00/pRadio_HW00.kicad_sch (KiCad schematic)
At the start: 10 parts, among them J1 PSoM_ESP32S2_Carrier_Board, J2 USB4510-03-1-A, J3 SJ2-3514A-SMT-TR, J4 S2B-PH-SM4-TB, SW1 450405020524, SW2 SW_Push, SW3 ACZ11BR1E-15FA1-20C, SW4 ACZ11BR1E-15FA1-20C, U1 SA818S

Commit message: Working on layout to see how compact it can get
Parts:
- SW2: footprint Component_lib:Kailh_socket_PG1350 -> Component_lib:SW_Kailh_Choc_V1
Changed lines of the file:
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@@
       (effects (font (size 1.27 1.27)))
     )
-    (property "Footprint" "Component_lib:Kailh_socket_PG1350" (at 66.04 157.48 0)
+    (property "Footprint" "Component_lib:SW_Kailh_Choc_V1" (at 66.04 157.48 0)
       (effects (font (size 1.27 1.27)) hide)
     )

Commit message: Created schematic
Parts:
- removed U1: SA818S, Component_lib:RF818, symbol Component_lib:SA818S
- added C1: 390n, symbol Component_lib:C
- added C10, C2, C4, C8: 100n, symbol Component_lib:C
- added C11, C14: 20p, symbol Component_lib:C
- added C12, C13: 36p, symbol Component_lib:C
- added C3, C7: 10p, symbol Component_lib:C
- added C5, C9: 2u2, symbol Component_lib:C
- added C6: 4u7, symbol Component_lib:C
- added IC1: LM4871MMX_NOPB, SOP65P490X110-8N, symbol Component_lib:LM4871MMX_NOPB
- added IC2: LM358D, SOIC127P600X175-8N, symbol Component_lib:LM358D
- added J5: U.FL-R-SMT-1_40_, UFLRSMT140, symbol Component_lib:U.FL-R-SMT-1_40_
- added L1, L3: 56n, symbol Component_lib:L
- added L2: 68n, symbol Component_lib:L
- added R1, R15, R3: 5k1, symbol Component_lib:R
- added R10, R12, R7, R8: 100k, symbol Component_lib:R
- added R11: 10, symbol Component_lib:R
- added R13, R14, R6: 0, symbol Component_lib:R
- added R2, R5: 20k, symbol Component_lib:R
- added R4: 10k, symbol Component_lib:R
- added R9: 6k, symbol Component_lib:R
- added U1: SA868S, Component_lib:RF818, symbol Component_lib:SA868S
- renumbered J2 to J1, J4 to J2, J1 to J4, SW4 to SW1, SW3 to SW2, SW1 to SW3, SW2 to SW4
Connections:
- net R_A: now reaches SW2.A
- net R_B: now reaches SW2.B
- net GND: now reaches SW2.C
- net GND: now also D1.1 (VSS), J1.A1 (GND), J1.A12 (GND), J1.B1 (GND), J1.B12 (GND), J1.MH1, J1.MH2, J1.MH3, J1.MH4, J2.2 (Pin_2), J2.MP (MountPin), J3.1 (SLEEVE), J4.1 (GND), J4.2 (GND), J4.22 (GND), J4.24 (GND), J4.41 (GND), J4.54 (GND), J4.59 (GND), J4.60 (GND), SW1.C, SW1.S2, SW2.S2, SW4.1, C10.1, C11.1, C12.1, C13.1, C14.1, C2.1, C3.2, C4.1, C5.1, C8.1, IC1.7 (GND), IC2.4 (V-), J5.2 (gnd), J5.3 (gnd), R1.2, R12.2, R3.2, R6.2, R8.1, U1.10 (GND), U1.9 (GND)
- net R_PB: now reaches SW2.S1
- net MIC: now reaches J3.3 (RING_1)
- net MIC: now also J4.37 (IO18/DAC), C6.1, R9.1
- net SPEAKER: now reaches J3.4 (RING_2)
- net SPEAKER: now also IC1.5 (VO1), R5.2
- net EXT_PTT: now reaches J3.A2 (TIP_1)
- net EXT_PTT: now also R14.2
- net EXT_MIC_DET: now reaches J3.B2 (TIP_2)
- net L_A: now reaches SW1.A
- net L_B: now reaches SW1.B
- net L_PB: now reaches SW1.S1
- net at J2.1 (Pin_1): now also SW3.3 (B)
- net VSYS: now reaches D1.2 (VDD)
- net VSYS: now also J4.14 (VSYS), J4.16 (VSYS), C10.2, U1.8 (VBAT)
- net LED_DATA: now reaches D1.3 (DIN)
- net PB_PTT: now reaches SW4.2
- net PB_PTT: now also R13.2
- net VBUS: now reaches J4.10 (VBUS)
- net VBUS: now also J1.A4 (VBUS), J1.A9 (VBUS), J1.B4 (VBUS), J1.B9 (VBUS), J4.12 (VBUS)
- net +3V3: now reaches J4.18 (3V3)
- net +3V3: now also J4.20 (3V3), C4.2, C8.2, IC1.6 (VDD), IC2.8 (V+), R15.2, R7.2, R9.2
- net AUDIO_IN: now reaches J4.39 (IO21)
- net AUDIO_IN: now also C1.1, U1.3 (Audio_OUT)
- net D+: now reaches J4.56 (D+)
- net D+: now also J1.A6 (D+), J1.B6 (D+)
- net D-: now reaches J4.58 (D-)
- net D-: now also J1.A7 (D-), J1.B7 (D-)
- net VBAT: now reaches J4.6 (VBAT)
- net VBAT: now also J4.8 (VBAT), SW3.1 (A)
- net at J1.A5 (CC1): now also R1.1
- net at J1.B5 (CC2): now also R3.1
- new net: C13.2, L2.2, L3.1
- new net: C12.2, L1.2, L2.1
- new net: C14.2, J5.1 (ant), L3.2
- new net: C9.1, R11.1
- new net: U1.11 (NC), U1.13 (NC), U1.14 (NC), U1.15 (NC), U1.2 (NC), U1.4 (NC)
- new net: C1.2, R2.1
- new net AMP_BYPASS: C2.2, IC1.2 (BYPASS)
- new net AMP_SHUTDOWN: IC1.1 (SHUTDOWN), R4.1
- new net MIC_AMPED: C9.2, R12.1, U1.18 (MIC_IN)
- new net MIC_AMP_+: C5.2, IC2.5 (IN2+), R7.1, R8.2
- new net MIC_AMP_-: C6.2, C7.1, IC2.6 (IN2-), R10.2
- new net MIC_AMP_OUT: C7.2, IC2.7 (OUT2), R10.1, R11.2
- new net POWERDOWN: R15.1, U1.6 (PD)
- new net SPK_AMP_IN: IC1.4 (-IN), R2.2, R5.1
- new net SPK_AMP_OUT_-: IC1.8 (VO2), R6.1
- new net SPK_AMP_VIN+: C3.1, IC1.3 (+IN)
- new net SQ: R4.2, U1.1 (Audio_ON)
- new net TX_POWER: U1.7 (H/L)
- new net VHF_ANT_OUT: C11.2, L1.1, U1.12 (ANT)
- new net VHF_PTT: R13.1, R14.1, U1.5 (PTT)
- new net VHF_RX: U1.16 (RXD)
- new net VHF_TX: U1.17 (TXD)
- no-connect marks 0 -> 19
Other:
- note added: "Close to pin 6"
- note added: "Close to pin 8"
- note added: "Connectors"
- note added: "Input mic amplifier"
- note added: "Output speaker amplifier"
- note added: "PSoM"
- note added: "RF low pass filter"
- note added: "User interface"
- note added: "VHF module"
- moved on the sheet: D1, J2, J3, J4, SW1, SW2, SW3, SW4

Commit message: Schematic done
Parts:
- C400: renamed from C10; footprint (none) -> Capacitor_SMD:C_0402_1005Metric
- C401: renamed from C11; footprint (none) -> Capacitor_SMD:C_0402_1005Metric
- C402: renamed from C12; footprint (none) -> Capacitor_SMD:C_0402_1005Metric
- C403: renamed from C13; footprint (none) -> Capacitor_SMD:C_0402_1005Metric
- C404: renamed from C14; footprint (none) -> Capacitor_SMD:C_0402_1005Metric
- C500: renamed from C1; footprint (none) -> Capacitor_SMD:C_0603_1608Metric
- C501: renamed from C3; footprint (none) -> Capacitor_SMD:C_0402_1005Metric
- C502: renamed from C2; footprint (none) -> Capacitor_SMD:C_0402_1005Metric
- C503: renamed from C4; footprint (none) -> Capacitor_SMD:C_0402_1005Metric
- C600: renamed from C5; footprint (none) -> Capacitor_SMD:C_0603_1608Metric
- C601: renamed from C6; footprint (none) -> Capacitor_SMD:C_0603_1608Metric
- C602: renamed from C7; footprint (none) -> Capacitor_SMD:C_0402_1005Metric
- C603: renamed from C9; footprint (none) -> Capacitor_SMD:C_0603_1608Metric
- C604: renamed from C8; footprint (none) -> Capacitor_SMD:C_0402_1005Metric
- IC500: renamed from IC1; footprint SOP65P490X110-8N -> Component_lib:SOP65P490X110-8N
- IC600: renamed from IC2; footprint SOIC127P600X175-8N -> Component_lib:SOIC127P600X175-8N
- J400: renamed from J5; footprint UFLRSMT140 -> Component_lib:u.fl
- L400: renamed from L1; footprint (none) -> Inductor_SMD:L_0402_1005Metric
- L401: renamed from L2; footprint (none) -> Inductor_SMD:L_0402_1005Metric
- L402: renamed from L3; footprint (none) -> Inductor_SMD:L_0402_1005Metric
- R100: renamed from R1; footprint (none) -> Resistor_SMD:R_0201_0603Metric
- R101: renamed from R3; footprint (none) -> Resistor_SMD:R_0201_0603Metric
- R400: renamed from R15; footprint (none) -> Resistor_SMD:R_0201_0603Metric
- R401: renamed from R13; footprint (none) -> Resistor_SMD:R_0201_0603Metric
- R402: renamed from R14; footprint (none) -> Resistor_SMD:R_0201_0603Metric
- R500: renamed from R5; footprint (none) -> Resistor_SMD:R_0201_0603Metric
- R501: renamed from R2; footprint (none) -> Resistor_SMD:R_0201_0603Metric
- R502: renamed from R4; footprint (none) -> Resistor_SMD:R_0201_0603Metric
- R503: renamed from R6; footprint (none) -> Resistor_SMD:R_0201_0603Metric
- R600: renamed from R7; footprint (none) -> Resistor_SMD:R_0402_1005Metric
- R601: renamed from R8; footprint (none) -> Resistor_SMD:R_0402_1005Metric
- R602: renamed from R9; footprint (none) -> Resistor_SMD:R_0402_1005Metric
- R603: renamed from R11; footprint (none) -> Resistor_SMD:R_0402_1005Metric
- R604: renamed from R12; footprint (none) -> Resistor_SMD:R_0402_1005Metric
- R605: renamed from R10; footprint (none) -> Resistor_SMD:R_0402_1005Metric
- renumbered D1 to D300, J1 to J100, J3 to J101, J2 to J102, J4 to J200, SW3 to SW100, SW1 to SW300, SW2 to SW301, SW4 to SW302, U1 to U400
Connections:
- net AUDIO_IN: now also J200.37 (IO18/DAC); no longer J200.39 (IO21)
- net EXT_MIC_DET: now also J200.29 (IO14)
- net EXT_PTT: now also J200.31 (IO15)
- net LED_DATA: now also J200.7 (IO3)
- net L_A: now also J200.15 (IO7)
- net L_B: now also J200.17 (IO8)
- net L_PB: now also J200.19 (IO9)
- net MIC: now also J200.35 (IO17/DAC); no longer J200.37 (IO18/DAC)
- net PB_PTT: now also J200.27 (IO13)
- net POWERDOWN: now also J200.11 (IO5)
- net PTT: now also J200.33 (IO16)
- net R_A: now also J200.21 (IO10)
- net R_B: now also J200.23 (IO11)
- net R_PB: now also J200.25 (IO12)
- net SQ: now also J200.13 (IO6)
- net TX_POWER: now also J200.9 (IO4)
- net CC1: now reaches J100.A5 (CC1), R100.1
- net CC2: now reaches J100.B5 (CC2), R101.1

Commit message: Working on routing
Parts:
- removed J100: USB4510-03-1-A, Component_lib:USB4510031A, symbol Component_lib:USB4510-03-1-A
- removed R100, R101: 5k1, Resistor_SMD:R_0201_0603Metric, symbol Component_lib:R
- renumbered J101 to J100, J102 to J101
Connections:
- net AUDIO_IN: now also J200.35 (IO17/DAC); no longer J200.37 (IO18/DAC)
- net EXT_MIC_DET: now also J200.52 (IO42); no longer J200.29 (IO14)
- net EXT_PTT: now also J200.5 (IO2); no longer J200.31 (IO15)
- net GND: now also SW300.MH1, SW300.MH2, SW301.MH1, SW301.MH2
- net LED_DATA: now also J200.46 (IO40); no longer J200.7 (IO3)
- net L_A: now also J200.27 (IO13); no longer J200.15 (IO7)
- net L_B: now also J200.25 (IO12); no longer J200.17 (IO8)
- net L_PB: now also J200.23 (IO11); no longer J200.19 (IO9)
- net MIC: now also J200.37 (IO18/DAC); no longer J200.35 (IO17/DAC)
- net PB_PTT: now also J200.7 (IO3); no longer J200.27 (IO13)
- net POWERDOWN: now also J200.9 (IO4); no longer J200.11 (IO5)
- net R_A: now also J200.19 (IO9); no longer J200.21 (IO10)
- net R_B: now also J200.21 (IO10); no longer J200.23 (IO11)
- net R_PB: now also J200.17 (IO8); no longer J200.25 (IO12)
- net SQ: now also J200.29 (IO14); no longer J200.13 (IO6)
- net TX_POWER: now also J200.11 (IO5); no longer J200.9 (IO4)
- net VHF_RX: now also J200.13 (IO6)
- net VHF_TX: now also J200.15 (IO7)
- net VBAT_IN: now reaches J101.1 (Pin_1), SW100.3 (B)
- net PTT: no longer names the net of J200.33 (IO16)
- no-connect marks 19 -> 17
Other:
- moved on the sheet: J100, J101, R401, R402, SW100
